File: ThermoBoard.kicad_pcb (KiCad board)
At the start: 4 copper layers, 0 parts

Commit message: Some changes to power circuitry, more layout
Parts:
- added C100: 10u, Capacitor_SMD:C_0603_1608Metric, F.Cu at (57.2, 124.5)
- added C101: 100n, Capacitor_SMD:C_0402_1005Metric, F.Cu at (66.5, 124.5)
- added C102: 10p, Capacitor_SMD:C_0402_1005Metric, F.Cu at (130.0, 100.8)
- added C103: 100n, Capacitor_SMD:C_0402_1005Metric, F.Cu at (130.0, 98.3)
- added C104: 100n, Capacitor_SMD:C_0402_1005Metric, F.Cu at (134.7, 95.0)
- added C105: 10p, Capacitor_SMD:C_0402_1005Metric, F.Cu at (130.0, 103.5)
- added C106: 100n, Capacitor_SMD:C_0402_1005Metric, F.Cu at (145.0, 97.5)
- added C107: 2u2, Capacitor_SMD:C_0603_1608Metric, F.Cu at (47.7, 20.6)
- added C108: 100n, Capacitor_SMD:C_0402_1005Metric, F.Cu at (143.0, 111.0)
- added C109: 2u2, Capacitor_SMD:C_0603_1608Metric, F.Cu at (47.7, 22.4)
- added C110: 100n, Capacitor_SMD:C_0402_1005Metric, F.Cu at (136.3, 111.0)
- added C111: 100n, Capacitor_SMD:C_0402_1005Metric, F.Cu at (130.0, 105.6)
- added C112: 1u, Capacitor_SMD:C_0603_1608Metric, F.Cu at (151.5, 88.8)
- added C113: 1u, Capacitor_SMD:C_0603_1608Metric, F.Cu at (152.0, 96.0)
- added C114: 1u, Capacitor_SMD:C_0603_1608Metric, F.Cu at (155.8, 91.0)
- added C115: 1u, Capacitor_SMD:C_0603_1608Metric, F.Cu at (152.0, 94.2)
- added C116: 100n, Capacitor_SMD:C_0402_1005Metric, F.Cu at (158.5, 100.0)
- added C117: 1u, Capacitor_SMD:C_0603_1608Metric, F.Cu at (158.2, 91.0)
- added C200: 5p6, Capacitor_SMD:C_0402_1005Metric, F.Cu at (133.4, 132.7)
- added C201: 5p6, Capacitor_SMD:C_0402_1005Metric, F.Cu at (133.4, 134.3)
- added C202: 10u, Capacitor_SMD:C_0603_1608Metric, F.Cu at (122.0, 156.1)
- added C203: 100n, Capacitor_SMD:C_0402_1005Metric, F.Cu at (133.4, 135.9)
- added C204: 100n, Capacitor_SMD:C_0402_1005Metric, F.Cu at (133.4, 137.6)
- added C205: 100n, Capacitor_SMD:C_0402_1005Metric, F.Cu at (133.4, 139.2)
- added C206: 100n, Capacitor_SMD:C_0402_1005Metric, F.Cu at (133.4, 140.9)
- added C207: 10p, Capacitor_SMD:C_0402_1005Metric, F.Cu at (133.4, 142.6)
- added C208: 22n, Capacitor_SMD:C_0402_1005Metric, F.Cu at (133.4, 144.2)
- added C209: 10p, Capacitor_SMD:C_0402_1005Metric, F.Cu at (135.7, 132.7)
- added C210: 10p, Capacitor_SMD:C_0402_1005Metric, F.Cu at (135.7, 134.3)
- added C211: 10p, Capacitor_SMD:C_0402_1005Metric, F.Cu at (135.7, 135.9)
- added C212: 100n, Capacitor_SMD:C_0402_1005Metric, F.Cu at (135.7, 137.6)
- added C300: 10n, Capacitor_SMD:C_0402_1005Metric, F.Cu at (35.5, 70.2)
- added C301: 100n, Capacitor_SMD:C_0402_1005Metric, F.Cu at (34.0, 65.7)
- added C302: 10n, Capacitor_SMD:C_0402_1005Metric, F.Cu at (35.5, 61.8)
- added C303: 10n, Capacitor_SMD:C_0402_1005Metric, F.Cu at (50.0, 72.3)
- added C304: 100n, Capacitor_SMD:C_0402_1005Metric, F.Cu at (64.0, 69.5)
- added C305: 10n, Capacitor_SMD:C_0402_1005Metric, F.Cu at (64.0, 71.2)
- added C306: 100n, Capacitor_SMD:C_0402_1005Metric, F.Cu at (37.0, 70.3)
- added C307: 100n, Capacitor_SMD:C_0402_1005Metric, F.Cu at (64.0, 74.5)
- added C308: 100n, Capacitor_SMD:C_0402_1005Metric, F.Cu at (60.0, 63.0)
- added C309: 100n, Capacitor_SMD:C_0402_1005Metric, F.Cu at (64.8, 62.0)
- added C310: 10n, Capacitor_SMD:C_0402_1005Metric, F.Cu at (66.2, 66.2)
- added C311: 100n, Capacitor_SMD:C_0402_1005Metric, F.Cu at (66.2, 67.9)
- added C312: 10n, Capacitor_SMD:C_0402_1005Metric, F.Cu at (66.2, 69.5)
- added C313: 10n, Capacitor_SMD:C_0402_1005Metric, F.Cu at (66.2, 71.2)
- added C314: 100n, Capacitor_SMD:C_0402_1005Metric, F.Cu at (66.2, 72.8)
- added C315: 10n, Capacitor_SMD:C_0402_1005Metric, F.Cu at (66.2, 74.5)
- added C316: 100n, Capacitor_SMD:C_0402_1005Metric, F.Cu at (63.0, 65.0)
- added C317: 100n, Capacitor_SMD:C_0402_1005Metric, F.Cu at (68.5, 64.6)
- added C318: 100n, Capacitor_SMD:C_0402_1005Metric, F.Cu at (68.5, 66.2)
- added C319: 100n, Capacitor_SMD:C_0402_1005Metric, F.Cu at (68.5, 67.9)
- added C400: 100n, Capacitor_SMD:C_0402_1005Metric, F.Cu at (172.7, 137.6)
- added C401: 100n, Capacitor_SMD:C_0402_1005Metric, F.Cu at (172.7, 139.3)
- added C402: 10u, Capacitor_SMD:C_0603_1608Metric, F.Cu at (180.2, 144.3)
- added C403: 10u, Capacitor_SMD:C_0603_1608Metric, F.Cu at (180.2, 146.0)
- added D100: PESD3V3, Diode_SMD:D_SOD-323, F.Cu at (48.3, 38.3)
- added D101: PESD3V3, Diode_SMD:D_SOD-323, F.Cu at (48.3, 41.2)
- added D102: PESD3V3, Diode_SMD:D_SOD-323, F.Cu at (48.3, 44.2)
- added D103: PESD3V3, Diode_SMD:D_SOD-323, F.Cu at (48.3, 47.1)
- added D104: PESD3V3, Diode_SMD:D_SOD-323, F.Cu at (48.2, 50.5)
- added D105: 1N4148WT, Diode_SMD:D_SOD-523, F.Cu at (152.0, 97.8)
- added D106: LED, LED_SMD:LED_0402_1005Metric, F.Cu at (157.2, 93.3)
- added D300: LED, LED_SMD:LED_0402_1005Metric, F.Cu at (39.0, 60.7)
- added D301: LED, LED_SMD:LED_0402_1005Metric, F.Cu at (68.5, 71.2)
- added D302: LED, LED_SMD:LED_0402_1005Metric, F.Cu at (68.5, 72.8)
- added D303: LED, LED_SMD:LED_0402_1005Metric, F.Cu at (68.5, 74.5)
- added D400: ESDCAN24-2BLY, Package_TO_SOT_SMD:SOT-23-3, F.Cu at (176.4, 145.8)
- added F100: 300mA, Capacitor_SMD:C_0603_1608Metric, F.Cu at (152.0, 99.6)
- added FB100: 120R, Capacitor_SMD:C_0603_1608Metric, F.Cu at (157.0, 88.3)
- added J100: Conn_01x05_Pin, Connector_PinHeader_2.54mm:PinHeader_1x05_P2.54mm_Vertical, F.Cu at (39.8, 30.2)
- added J101: Conn_01x03, Connector_PinHeader_2.54mm:PinHeader_1x03_P2.54mm_Vertical, F.Cu at (39.8, 45.0)
- added J102: TC2030, Connector:Tag-Connect_TC2030-IDC-NL_2x03_P1.27mm_Vertical, F.Cu at (57.5, 48.5)
- added J103: Screw_Terminal_01x02, TerminalBlock_Phoenix:TerminalBlock_Phoenix_MPT-0,5-2-2.54_1x02_P2.54mm_Horizontal, F.Cu at (164.5, 115.5)
- added J104: USB_C_Receptacle_USB2.0_16P, Connector_USB:USB_C_Receptacle_HRO_TYPE-C-31-M-12, F.Cu at (167.0, 103.0)
- added J200: RJ45_Hanrun_HR911105A_Horizontal, Connector_RJ:RJ45_Hanrun_HR911105A_Horizontal, F.Cu at (116.4, 136.1)
- added J300: Conn_01x02_Pin, Connector_PinHeader_2.54mm:PinHeader_1x02_P2.54mm_Vertical, F.Cu at (30.0, 67.3)
- added J301: Conn_01x02_Pin, Connector_PinHeader_2.54mm:PinHeader_1x02_P2.54mm_Vertical, F.Cu at (69.7, 57.3)
- added J302: Conn_01x02_Pin, Connector_PinHeader_2.54mm:PinHeader_1x02_P2.54mm_Vertical, F.Cu at (74.3, 57.3)
- added J303: Conn_01x02_Pin, Connector_PinHeader_2.54mm:PinHeader_1x02_P2.54mm_Vertical, F.Cu at (78.9, 57.3)
- added J400: Conn_01x04_Pin, Connector_PinHeader_2.54mm:PinHeader_1x04_P2.54mm_Vertical, F.Cu at (168.5, 138.7)
- added JP200: Jumper_2_Bridged, Jumper:SolderJumper-2_P1.3mm_Bridged_Pad1.0x1.5mm, F.Cu at (125.1, 149.5)
- added L100: 10n, Inductor_SMD:L_0603_1608Metric, F.Cu at (154.8, 95.0)
- added R100: 10k, Resistor_SMD:R_0402_1005Metric, F.Cu at (43.1, 20.5)
- added R101: 10k, Resistor_SMD:R_0402_1005Metric, F.Cu at (43.1, 22.1)
- added R102: 49R9, Resistor_SMD:R_0402_1005Metric, F.Cu at (43.1, 23.8)
- added R103: 49R9, Resistor_SMD:R_0402_1005Metric, F.Cu at (43.1, 25.4)
- added R104: 49R9, Resistor_SMD:R_0402_1005Metric, F.Cu at (43.1, 27.1)
- added R105: 49R9, Resistor_SMD:R_0402_1005Metric, F.Cu at (45.4, 18.9)
- added R106: 0R, Resistor_SMD:R_0402_1005Metric, F.Cu at (163.5, 97.0)
- added R107: 5k1, Resistor_SMD:R_0402_1005Metric, F.Cu at (160.5, 101.0)
- added R108: 5k1, Resistor_SMD:R_0402_1005Metric, F.Cu at (160.5, 104.5)
- added R109: 330R, Resistor_SMD:R_0402_1005Metric, F.Cu at (157.2, 94.3)
- added R200: 33R, Resistor_SMD:R_0402_1005Metric, F.Cu at (135.7, 139.2)
- added R201: 33R, Resistor_SMD:R_0402_1005Metric, F.Cu at (135.7, 140.9)
- added R202: 10k, Resistor_SMD:R_0402_1005Metric, F.Cu at (135.7, 142.6)
- added R203: 33R, Resistor_SMD:R_0402_1005Metric, F.Cu at (135.7, 144.2)
- added R204: 10k, Resistor_SMD:R_0402_1005Metric, F.Cu at (137.9, 132.7)
- added R205: 10k, Resistor_SMD:R_0402_1005Metric, F.Cu at (137.9, 134.3)
- added R206: 10k, Resistor_SMD:R_0402_1005Metric, F.Cu at (137.9, 135.9)
- added R207: 10k, Resistor_SMD:R_0402_1005Metric, F.Cu at (137.9, 137.6)
- added R208: 10k, Resistor_SMD:R_0402_1005Metric, F.Cu at (137.9, 139.2)
- added R209: 10k, Resistor_SMD:R_0402_1005Metric, F.Cu at (137.9, 140.9)
- added R210: 12k1, Resistor_SMD:R_0402_1005Metric, F.Cu at (137.9, 142.6)
- added R211: 49R9, Resistor_SMD:R_0402_1005Metric, F.Cu at (137.9, 144.2)
- added R212: 0R, Resistor_SMD:R_0402_1005Metric, F.Cu at (140.2, 132.7)
- added R213: 49R9, Resistor_SMD:R_0402_1005Metric, F.Cu at (140.2, 134.3)
- added R214: 49R9, Resistor_SMD:R_0402_1005Metric, F.Cu at (140.2, 135.9)
- added R215: 49R9, Resistor_SMD:R_0402_1005Metric, F.Cu at (140.2, 137.6)
- added R216: 0R, Resistor_SMD:R_0402_1005Metric, F.Cu at (140.2, 139.2)
- added R217: 330R, Resistor_SMD:R_0402_1005Metric, F.Cu at (140.2, 140.9)
- added R218: 330R, Resistor_SMD:R_0402_1005Metric, F.Cu at (140.2, 142.6)
- added R300: 0R, Resistor_SMD:R_0603_1608Metric, F.Cu at (34.0, 68.4)
- added R301: 0R, Resistor_SMD:R_0603_1608Metric, F.Cu at (34.0, 63.1)
- added R302: 0R, Resistor_SMD:R_0603_1608Metric, F.Cu at (73.1, 66.5)
- added R303: 0R, Resistor_SMD:R_0603_1608Metric, F.Cu at (73.1, 68.2)
- added R304: 0R, Resistor_SMD:R_0603_1608Metric, F.Cu at (37.0, 61.1)
- added R305: 0R, Resistor_SMD:R_0603_1608Metric, F.Cu at (75.5, 64.8)
- added R306: 10k, Resistor_SMD:R_0402_1005Metric, F.Cu at (64.0, 58.0)
- added R307: 10k, Resistor_SMD:R_0402_1005Metric, F.Cu at (71.0, 63.0)
- added R308: 330R, Resistor_SMD:R_0402_1005Metric, F.Cu at (40.5, 60.7)
- added R309: 330R, Resistor_SMD:R_0402_1005Metric, F.Cu at (70.7, 67.9)
- added R310: 0R, Resistor_SMD:R_0603_1608Metric, F.Cu at (75.5, 66.5)
- added R311: 0R, Resistor_SMD:R_0603_1608Metric, F.Cu at (75.5, 68.2)
- added R312: 0R, Resistor_SMD:R_0603_1608Metric, F.Cu at (78.0, 63.0)
- added R313: 0R, Resistor_SMD:R_0603_1608Metric, F.Cu at (78.0, 64.8)
- added R314: 0R, Resistor_SMD:R_0603_1608Metric, F.Cu at (78.0, 66.5)
- added R315: 0R, Resistor_SMD:R_0603_1608Metric, F.Cu at (78.0, 68.2)
- added R316: 10k, Resistor_SMD:R_0402_1005Metric, F.Cu at (70.7, 69.5)
- added R317: 10k, Resistor_SMD:R_0402_1005Metric, F.Cu at (70.7, 71.2)
- added R318: 330R, Resistor_SMD:R_0402_1005Metric, F.Cu at (70.7, 72.8)
- added R319: 330R, Resistor_SMD:R_0402_1005Metric, F.Cu at (70.7, 74.5)
- added R400: 10k, Resistor_SMD:R_0402_1005Metric, F.Cu at (172.7, 140.9)
- added R401: 49R9, Resistor_SMD:R_0402_1005Metric, F.Cu at (172.7, 142.6)
- added R402: 49R9, Resistor_SMD:R_0402_1005Metric, F.Cu at (172.7, 144.2)
- added R403: 60R, Resistor_SMD:R_0402_1005Metric, F.Cu at (172.7, 145.9)
- added R404: 60R, Resistor_SMD:R_0402_1005Metric, F.Cu at (172.7, 147.5)
- added SW100: SW_Push, Button_Switch_SMD:SW_SPST_B3S-1000, F.Cu at (28.6, 47.2)
- added TP100: +5V, TestPoint:TestPoint_Pad_D2.0mm, F.Cu at (20.5, 26.5)
- added TP101: +VIN, TestPoint:TestPoint_Pad_D2.0mm, F.Cu at (20.5, 29.9)
- added TP102: +3V3, TestPoint:TestPoint_Pad_D2.0mm, F.Cu at (20.5, 34.0)
- added TP103: +3.3VA, TestPoint:TestPoint_Pad_D2.0mm, F.Cu at (20.5, 38.0)
- added U100: STM32H563RITx, Package_QFP:LQFP-64_10x10mm_P0.5mm, F.Cu at (139.0, 103.5)
- added U101: AP2112K-3.3, Package_TO_SOT_SMD:SOT-23-5, F.Cu at (152.2, 91.3)
- added U102: USBLC6-2SC6, Package_TO_SOT_SMD:SOT-23-6, F.Cu at (157.0, 102.5)
- added U200: LAN8742A, Package_DFN_QFN:VQFN-24-1EP_4x4mm_P0.5mm_EP2.5x2.5mm_ThermalVias, F.Cu at (135.4, 148.2)
- added U201: USBLC6-4SC6, Package_TO_SOT_SMD:SOT-23-6, F.Cu at (134.8, 153.7)
- added U300: MAX31856, Package_SO:TSSOP-14_4.4x5mm_P0.65mm, F.Cu at (39.0, 65.7)
- added U301: MAX31856, Package_SO:TSSOP-14_4.4x5mm_P0.65mm, F.Cu at (72.0, 97.0)
- added U302: MAX31856, Package_SO:TSSOP-14_4.4x5mm_P0.65mm, F.Cu at (36.0, 88.0)
- added U303: MAX31856, Package_SO:TSSOP-14_4.4x5mm_P0.65mm, F.Cu at (54.0, 93.0)
- added U400: TJA1042T-3, Package_SO:SOIC-8_3.9x4.9mm_P1.27mm, F.Cu at (191.5, 144.3)
- added Y100: 16MHz, Crystal:Crystal_SMD_EuroQuartz_MJ-4Pin_5.0x3.2mm, F.Cu at (125.0, 102.0)
- added Y200: 25MHz, Library:CRYSTAL-SMD_4P-L2.0-W1.6-BL, F.Cu at (118.8, 156.9)
Routing:
- net /Microcontroller/USB_CONN_CC2: track 0.00 -> 2.06 mm
- net /Microcontroller/USB_CONN_CC1: track 0.00 -> 2.06 mm
Other:
- board text added: "${REFERENCE}"
- board text added: "+"
- board text added: "-"

Commit message: Some more schematic updates
Parts:
- moved R302 58.9 mm to (24.0, 99.0), turned to 90 degrees
- moved J301 46.3 mm to (30.0, 81.0)
- moved R310 45.4 mm to (34.0, 84.8), turned to 90 degrees
- moved R311 42.9 mm to (34.0, 79.2), turned to -90 degrees
- moved R314 42.3 mm to (37.0, 77.2), turned to -90 degrees
- moved C310 36.5 mm to (35.5, 86.0), turned to 90 degrees
- moved C311 35.2 mm to (34.0, 82.0), turned to 90 degrees
- moved C318 33.4 mm to (41.5, 86.0), turned to -90 degrees
- moved C316 33.4 mm to (37.0, 86.0), turned to -90 degrees
- moved U301 33.0 mm to (39.0, 98.5)
- moved C312 31.9 mm to (35.5, 78.0), turned to 90 degrees
- moved R318 30.4 mm to (40.5, 76.5), turned to 90 degrees
- moved D302 29.2 mm to (39.5, 76.5), turned to 90 degrees
- moved U303 26.2 mm to (39.0, 114.5)
- moved C308 19.9 mm to (41.5, 70.2)
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Routing:
- net /Microcontroller/USB_CONN_CC2: track 2.06 -> 0.00 mm
- net /Microcontroller/USB_CONN_CC1: track 2.06 -> 0.00 mm
Other:
- board text added: "CAN"

Commit message: Extremely incomplete, preliminary, pre-alpha, ugly layout
Parts:
- removed the C207 at (133.4, 142.6)
- removed C209, C210, C211: 10p, Capacitor_SMD:C_0402_1005Metric
- added H200: MountingHole, MountingHole:MountingHole_3.2mm_M3, F.Cu at (110.0, 85.0)
- added H201: MountingHole, MountingHole:MountingHole_3.2mm_M3, F.Cu at (166.0, 85.0)
- added H202: MountingHole, MountingHole:MountingHole_3.2mm_M3, F.Cu at (166.0, 135.0)
- added H203: MountingHole, MountingHole:MountingHole_3.2mm_M3, F.Cu at (3.48, 3.48)
- C107, C109: footprint Capacitor_SMD:C_0603_1608Metric -> Capacitor_SMD:C_0402_1005Metric
- TP102: footprint TestPoint:TestPoint_Pad_D2.0mm -> TestPoint:TestPoint_Pad_D1.0mm
- moved TP101 155.0 mm to (160.0, 97.5)
- moved TP103 148.7 mm to (160.0, 89.5)
- moved TP100 145.4 mm to (148.8, 95.0)
- moved TP102 143.9 mm to (153.7, 88.5)
- moved C107 130.9 mm to (142.0, 111.5), turned to -90 degrees
- moved R306 130.1 mm to (163.9, 71.0), turned to 180 degrees
- moved J300 129.8 mm to (159.8, 67.0), turned to 90 degrees
- moved C308 129.7 mm to (164.7, 72.5), turned to 0 degrees
- moved R308 129.0 mm to (165.3, 74.0), turned to 180 degrees
- moved D300 127.8 mm to (166.3, 76.8), turned to 0 degrees
- moved C306 127.2 mm to (161.1, 71.0), turned to 0 degrees
- moved R300 126.9 mm to (166.3, 77.8), turned to 0 degrees
- moved R304 124.3 mm to (158.2, 71.0), turned to 0 degrees
- moved U300 122.2 mm to (160.8, 76.0), turned to -90 degrees
- moved C304 120.8 mm to (156.3, 72.5), turned to 0 degrees
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- renumbered C208 to C207, C212 to C208, C306 to C300, C308 to C301, C316 to C302, C318 to C303, C300 to C304, C310 to C305, C301 to C306, C311 to C307, C302 to C308, C312 to C309, C307 to C310, C309 to C311, C317 to C312, C319 to C313, C303 to C314, C313 to C315, C304 to C316, C314 to C317, C305 to C318, C315 to C319, D302 to D301, D301 to D302, J302 to J301, J301 to J302, R308 to R300, R318 to R301, R306 to R302, R316 to R303, R300 to R304, R310 to R305, R301 to R306, R311 to R307, R304 to R308, R314 to R309, R309 to R310, R319 to R311, R307 to R312, R317 to R313, R302 to R314, R312 to R315, R303 to R316, R313 to R317, R305 to R318, R315 to R319, U302 to U301, U301 to U302
Connections:
- C100 pad 1: +3.3V -> +3V3
- C103 pad 1: +3.3V -> +3V3
- C104 pad 1: +3.3V -> +3V3
- C106 pad 1: +3.3V -> +3V3
- C108 pad 1: +3.3V -> +3V3
- C110 pad 1: +3.3V -> +3V3
- C111 pad 1: +3.3V -> +3V3
- J101 pad 3: +3.3V -> +3V3
- R100 pad 1: +3.3V -> +3V3
- R302 pad 1: +3.3V -> +3V3
- R303 pad 1: +3.3V -> +3V3
- R312 pad 1: +3.3V -> +3V3
- R313 pad 1: +3.3V -> +3V3
- U100 pad 1: +3.3V -> +3V3
- U100 pad 13: +3.3V -> +3V3
- U100 pad 19: +3.3V -> +3V3
- U100 pad 32: +3.3V -> +3V3
- U100 pad 48: +3.3V -> +3V3
- U100 pad 64: +3.3V -> +3V3
- U201 pad 1: /Ethernet/TX+ -> /Ethernet/TX-
- U201 pad 3: /Ethernet/TX- -> /Ethernet/TX+
Routing:
- net +3V3: track 0.00 -> 357.7 mm, vias 0 -> 24
- net SPI_SCK: track 0.00 -> 104.4 mm, vias 0 -> 5
- net SPI_MOSI: track 0.00 -> 95.6 mm
- net +3.3VA: track 0.00 -> 92.2 mm, vias 0 -> 2
- net SPI_MISO: track 0.00 -> 86.5 mm, vias 0 -> 5
- net NDRDY4: track 0.00 -> 72.5 mm, vias 0 -> 2
- net +5V: track 0.00 -> 68.2 mm, vias 0 -> 3
- net NDRDY3: track 0.00 -> 61.9 mm, vias 0 -> 2
- net NRST: track 0.00 -> 59.4 mm, vias 0 -> 3
- net NDRDY2: track 0.00 -> 54.4 mm, vias 0 -> 2
- net NFAULT3: track 0.00 -> 51.7 mm, vias 0 -> 4
- net SPI_CS4: track 0.00 -> 50.7 mm, vias 0 -> 6
- net NFAULT4: track 0.00 -> 49.1 mm, vias 0 -> 4
- net NFAULT1: track 0.00 -> 48.0 mm, vias 0 -> 2
- net NFAULT2: track 0.00 -> 42.0 mm, vias 0 -> 2
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- added copper zone on F.Cu, net GND
- added copper zone on In1.Cu, net GND
- added copper zone on In2.Cu, net GND
Other:
- board outline added: 66 x 75 mm
- board text added: "+3V3"
- board text added: "BOOT"
- board text added: "GND"
- board text added: "NRST"
- board text added: "RESET"
- board text added: "SWCLK"
- board text added: "SWDIO"
- board text added: "T1"
- board text added: "T2"
- board text added: "T3"
- board text added: "T4"
- board text removed: "CAN"
